File: HARDWARE/LumiDrive.brd (EAGLE design)
At the start: 33 x 57 mm, 94 parts, among them Q1 2.5A/30V/105mΩ, U1 MCP73831, U2 ATSAMD21G-A, U3 3.3V, U4 W25Q32FV, Y1 32.768kHz

Commit message: Ready for protos round 2 (round 1 for me)
Parts:
- removed J6: (no value), SparkFun-Connectors:1X02_NO_SILK
- removed J7: (no value), SparkFun-Connectors:1X06_NO_SILK
- removed U$25: (no value), LumiDrive:LUMIDRIVE0
- removed U$33, U$7: (no value), Labels:GND-04
- removed U$34: (no value), RED2:RED0
- removed U$35: (no value), YLW2:YLW0
- removed U$36: (no value), INPUT:INPUT0
- added J1: (no value), SparkFun-Connectors:1X02_NO_SILK
- added U$29: (no value), SCORP_SMALL:SILHOUETTE#OF#A#SCORPION#JPG
- J5: device SparkFun-Connectors:1X02_NO_SILK -> SparkFun-Connectors:1X06_NO_SILK
- LOGO1: value OSHW-LOGOMINI -> OSHW-LOGOM; device SparkFun-Aesthetics:OSHW-LOGO-MINI -> SparkFun-Aesthetics:OSHW-LOGO-M
- U$1: device INPUT:INPUT0 -> Labels:GND-04
- U$5: device RED2:RED0 -> Labels:GND-04
- U$6: device YLW2:YLW0 -> LumiDrive_SMALL:LUMIDRIVE0
- moved D3 36.1 mm to (26.4, 36.8), turned to 90 degrees
- moved LOGO1 32.1 mm to (29.6, 15.5)
- moved U$32 32.0 mm to (31.5, 49.5), turned to 0 degrees
- moved U$8 31.6 mm to (27.8, 49.5), turned to 0 degrees
- moved U$6 27.9 mm to (2.54, 19.1)
- moved U$28 25.9 mm to (29.6, 8.89), turned to 0 degrees
- moved U$5 22.2 mm to (31.5, 33.0), flipped to the bottom, turned to 0 degrees
- moved U$1 18.0 mm to (26.7, 33.0), turned to 0 degrees
- moved U$19 14.0 mm to (26.7, 47.0)
- moved U$26 14.0 mm to (31.5, 47.0)
- moved J5 11.7 mm to (31.8, 22.9), turned to 90 degrees
- moved LOGO3 11.4 mm to (16.0, 37.1)
- moved U$20 5.08 mm to (26.8, 35.6)
- moved U$27 5.08 mm to (31.5, 35.6)
- moved U$17 4.07 mm to (27.2, 46.1), turned to 270 degrees
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Connections:
- net 3.3V: now also J5.6; no longer J7.5
- net 5V: now also J1.1; no longer J5.2, J6.2
- net A3: now also J5.1; no longer J7.1
- net A4: now also J5.2; no longer J7.2
- net D8: now also J5.3; no longer J7.3
- net D9: now also J5.4; no longer J7.4
- net GND: now also J1.2, J5.5; no longer J5.1, J6.1, J7.6
- net VIN: now also J4.P2, J4.P4
- net V_BATT: no longer J4.P2, J4.P4
Routing:
- net V_BATT: track 66.6 -> 10.9 mm, vias 2 -> 0
- net VIN: track 9.44 -> 54.0 mm, vias 0 -> 2
- net V_USB: track 77.1 -> 44.0 mm
- net 5V: track 26.2 -> 15.6 mm, vias 1 -> 0
- net N$7: track 2.57 -> 6.26 mm, vias 0 -> 2
- net A4: track 20.7 -> 19.3 mm
- net A3: track 23.2 -> 21.8 mm
- net D9: track 16.3 -> 15.3 mm
- net D8: track 18.8 -> 18.1 mm
- net 3.3V: track 89.8 -> 90.2 mm, vias 1 -> 2
- net GND: vias 30 -> 34
