File: HARDWARE/LumiDrive.sch (EAGLE design)
At the start: 56 parts, among them Q1 2.5A/30V/105mΩ, U1 MCP73831, U2 ATSAMD21G-A, U3 3.3V, U4 W25Q32FV, Y1 32.768kHz

Commit message: Ready for protos round 2 (round 1 for me)
Parts:
- removed J6: (no value), SparkFun-Connectors:CONN_021X02_NO_SILK
- removed J7: (no value), SparkFun-Connectors:CONN_06NO_SILK_NO_POP
- added J1: (no value), SparkFun-Connectors:CONN_021X02_NO_SILK
- J5: device SparkFun-Connectors:CONN_021X02_NO_SILK -> SparkFun-Connectors:CONN_06NO_SILK_FEMALE_PTH
- LOGO1: value OSHW-LOGOMINI -> OSHW-LOGOM; device SparkFun-Aesthetics:OSHW-LOGOMINI -> SparkFun-Aesthetics:OSHW-LOGOM
Connections:
- net 3.3V: now also J5.6; no longer J7.5
- net 5V: now also J1.1; no longer J5.2, J6.2
- net A3: now also J5.1; no longer J7.1
- net A4: now also J5.2; no longer J7.2
- net D8: now also J5.3; no longer J7.3
- net D9: now also J5.4; no longer J7.4
- net GND: now also J1.2, J5.5; no longer J5.1, J6.1, J7.6
- net VIN: now also J4.2
- net V_BATT: no longer J4.2
Other:
- moved on the sheet: D9, R1

Commit message: Adds production files and assembly sheet, and fixes swapped lipo connector pads
Parts:
- removed J2: (no value), SparkFun-Connectors:CONN_02-JST-2MM-SMT
- added J6: (no value), SparkFun-Connectors:JST_2MM_MALE
- added TP6: TEST-POINT3X4, SparkFun-Connectors:TEST-POINT3X4
Connections:
- net GND: now also J6.-; no longer J2.1
- net V_BATT: now also J6.+, TP6.1; no longer J2.2
Changed lines of the file:
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@@
 <part name="C16" library="SparkFun-Capacitors" deviceset="15PF" device="-0603-50V-5%" value="15pF"/>
 <part name="GND34" library="SparkFun-PowerSymbols" deviceset="GND" device=""/>
-<part name="J2" library="SparkFun-Connectors" deviceset="CONN_02" device="-JST-2MM-SMT"/>
 <part name="GND1" library="SparkFun-PowerSymbols" deviceset="GND" device=""/>
 <part name="R1" library="SparkFun-Resistors" deviceset="1KOHM" device="-0603-1/10W-1%" value="1k"/>
@@
 <part name="SUPPLY14" library="SparkFun-PowerSymbols" deviceset="5V" device=""/>
 <part name="J5" library="SparkFun-Connectors" deviceset="CONN_06" device="NO_SILK_FEMALE_PTH"/>
+<part name="J6" library="SparkFun-Connectors" deviceset="JST_2MM_MALE" device=""/>
+<part name="TP6" library="SparkFun-Connectors" deviceset="TEST-POINT" device="3X4" value="TEST-POINT3X4"/>
 </parts>
 <sheets>
@@
 <attribute name="VALUE" x="17.78" y="45.466" size="1.778" layer="96" align="top-center"/>
 </instance>
-<instance part="J2" gate="G$1" x="58.42" y="162.56" smashed="yes">
-<attribute name="VALUE" x="55.88" y="157.734" size="1.778" layer="96" font="vector"/>
-<attribute name="NAME" x="55.88" y="168.148" size="1.778" layer="95" font="vector"/>
-</instance>
 <instance part="GND1" gate="1" x="203.2" y="106.68" smashed="yes">
 <attribute name="VALUE" x="203.2" y="106.426" size="1.778" layer="96" align="top-center"/>
@@
 <attribute name="VALUE" x="241.3" y="131.826" size="1.778" layer="96" font="vector" rot="R180"/>
 <attribute name="NAME" x="241.3" y="111.252" size="1.778" layer="95" font="vector" rot="R180"/>
+</instance>
+<instance part="J6" gate="G$1" x="60.96" y="162.56" smashed="yes" rot="R90">
+<attribute name="NAME" x="55.118" y="160.02" size="1.778" layer="95" rot="R90"/>
+</instance>
+<instance part="TP6" gate="G$1" x="71.12" y="165.1" smashed="yes">
+<attribute name="NAME" x="70.866" y="166.37" size="1.778" layer="95" font="vector"/>
 </instance>
 </instances>
@@
 <segment>
 <pinref part="U2" gate="G$1" pin="VDDIO@36"/>
-<wire x1="106.68" y1="81.28" x2="116.84" y2="81.28" width="0.1524" layer="91"/>
-<wire x1="116.84" y1="81.28" x2="116.84" y2="83.82" width="0.1524" layer="91"/>
-<wire x1="116.84" y1="83.82" x2="127" y2="83.82" width="0.1524" layer="91"/>
+<wire x1="106.68" y1="81.28" x2="109.22" y2="81.28" width="0.1524" layer="91"/>
+<wire x1="109.22" y1="81.28" x2="109.22" y2="83.82" width="0.1524" layer="91"/>
+<wire x1="109.22" y1="83.82" x2="127" y2="83.82" width="0.1524" layer="91"/>
 <pinref part="U2" gate="G$1" pin="VDDIO@17"/>
 <pinref part="C10" gate="G$1" pin="1"/>
@@
 <wire x1="127" y1="83.82" x2="127" y2="86.36" width="0.1524" layer="91"/>
 <wire x1="127" y1="86.36" x2="127" y2="88.9" width="0.1524" layer="91"/>
-<wire x1="106.68" y1="83.82" x2="116.84" y2="83.82" width="0.1524" layer="91"/>
-<junction x="116.84" y="83.82"/>
+<wire x1="106.68" y1="83.82" x2="109.22" y2="83.82" width="0.1524" layer="91"/>
+<junction x="109.22" y="83.82"/>
 <pinref part="C12" gate="G$1" pin="1"/>
 <wire x1="127" y1="86.36" x2="137.16" y2="86.36" width="0.1524" layer="91"/>
@@
 </segment>
 <segment>
-<pinref part="J2" gate="G$1" pin="1"/>
 <wire x1="66.04" y1="162.56" x2="68.58" y2="162.56" width="0.1524" layer="91"/>
 <pinref part="GND3" gate="1" pin="GND"/>
 <wire x1="68.58" y1="162.56" x2="68.58" y2="160.02" width="0.1524" layer="91"/>
+<pinref part="J6" gate="G$1" pin="-"/>
 </segment>
 <segment>
@@
 <net name="V_BATT" class="0">
 <segment>
-<pinref part="J2" gate="G$1" pin="2"/>
 <wire x1="66.04" y1="165.1" x2="68.58" y2="165.1" width="0.1524" layer="91"/>
 <wire x1="68.58" y1="165.1" x2="68.58" y2="167.64" width="0.1524" layer="91"/>
 <pinref part="SUPPLY4" gate="G$1" pin="V_BATT"/>
-</segment>
-<segment>
+<pinref part="J6" gate="G$1" pin="+"/>
+<pinref part="TP6" gate="G$1" pin="1"/>
+<wire x1="71.12" y1="165.1" x2="68.58" y2="165.1" width="0.1524" layer="91"/>
+<junction x="68.58" y="165.1"/>
+</segment>
+<segment>

Commit message: Adds testpoints to LED SLCK and MOSI lines, extra silk labels for INPUT and OUTPUT .....
 labeling INPUT as 3.3V-5V, deletes old production files
Parts:
- added TP7, TP8: TEST-POINT3X4, SparkFun-Connectors:TEST-POINT3X4
- FB1: device SparkFun-Inductors:FERRITE_BEAD-0603 -> SparkFun-Coils:INDUCTORFB-30OHM
Connections:
- net LED_MOSI: now also TP7.1
- net LED_SCK: now also TP8.1
Other:
- note added: "v10"
- note removed: "v02"
- moved on the sheet: C2
Changed lines of the file:
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@@
 <part name="GND5" library="SparkFun-PowerSymbols" deviceset="GND" device=""/>
 <part name="GND6" library="SparkFun-PowerSymbols" deviceset="GND" device=""/>
-<part name="FB1" library="SparkFun-Inductors" deviceset="FERRITE_BEAD" device="-0603" value="30Ω/1.8A"/>
+<part name="FB1" library="SparkFun-Coils" deviceset="INDUCTOR" device="FB-30OHM" value="30Ω/1.8A"/>
 <part name="GND2" library="SparkFun-PowerSymbols" deviceset="GND" device=""/>
 <part name="SUPPLY2" library="SparkFun-PowerSymbols" deviceset="3.3V" device=""/>
@@
 <part name="J6" library="SparkFun-Connectors" deviceset="JST_2MM_MALE" device=""/>
 <part name="TP6" library="SparkFun-Connectors" deviceset="TEST-POINT" device="3X4" value="TEST-POINT3X4"/>
+<part name="TP7" library="SparkFun-Connectors" deviceset="TEST-POINT" device="3X4" value="TEST-POINT3X4"/>
+<part name="TP8" library="SparkFun-Connectors" deviceset="TEST-POINT" device="3X4" value="TEST-POINT3X4"/>
 </parts>
 <sheets>
@@
 <text x="83.82" y="134.62" size="1.524" layer="97" font="vector">600mA out
 6V max in</text>
-<text x="238.76" y="10.16" size="2.54" layer="94" font="vector" align="top-left">v02</text>
+<text x="238.76" y="10.16" size="2.54" layer="94" font="vector" align="top-left">v10</text>
 <text x="172.72" y="13.716" size="2.54" layer="94" font="vector" align="top-left">Mike Hord</text>
 <text x="57.658" y="87.63" size="1.778" layer="97" font="vector">ATSAMD21G18
@@
 <text x="150.622" y="95.758" size="2.54" layer="94" font="vector" align="top-left">SPI Flash</text>
 <text x="3.302" y="95.758" size="2.54" layer="94" font="vector" align="top-left">ATSAMD21G18A</text>
-<text x="201.422" y="144.018" size="2.54" layer="94" font="vector" align="top-left">User LED and Header</text>
+<text x="197.358" y="145.034" size="2.54" layer="94" font="vector" align="top-left">User LED and Header</text>
 <wire x1="200.66" y1="147.32" x2="248.92" y2="147.32" width="0.2032" layer="97" style="shortdash"/>
 <wire x1="167.64" y1="147.32" x2="116.84" y2="147.32" width="0.2032" layer="97" style="shortdash"/>
@@
 <attribute name="VALUE" x="32.004" y="68.961" size="1.778" layer="96" font="vector"/>
 </instance>
-<instance part="C2" gate="G$1" x="7.62" y="12.7" smashed="yes">
-<attribute name="NAME" x="9.144" y="15.621" size="1.778" layer="95" font="vector"/>
-<attribute name="VALUE" x="9.144" y="10.541" size="1.778" layer="96" font="vector"/>
+<instance part="C2" gate="G$1" x="7.62" y="15.24" smashed="yes">
+<attribute name="NAME" x="9.144" y="18.161" size="1.778" layer="95" font="vector"/>
+<attribute name="VALUE" x="9.144" y="13.081" size="1.778" layer="96" font="vector"/>
 </instance>
 <instance part="C10" gate="G$1" x="127" y="76.2" smashed="yes">
@@
 <attribute name="PROD_ID" x="7.62" y="30.48" size="1.27" layer="96" display="off"/>
 <attribute name="NAME" x="8.89" y="33.02" size="1.778" layer="95" font="vector"/>
-<attribute name="VALUE" x="8.89" y="27.94" size="1.778" layer="96" font="vector" align="top-left"/>
-</instance>
-<instance part="GND2" gate="1" x="7.62" y="5.08" smashed="yes">
-<attribute name="VALUE" x="7.62" y="4.826" size="1.778" layer="96" align="top-center"/>
-</instance>
-<instance part="SUPPLY2" gate="G$1" x="7.62" y="40.64" smashed="yes">
-<attribute name="VALUE" x="7.62" y="43.434" size="1.778" layer="96" align="bottom-center"/>
+</instance>
+<instance part="GND2" gate="1" x="7.62" y="7.62" smashed="yes">
+<attribute name="VALUE" x="7.62" y="7.366" size="1.778" layer="96" align="top-center"/>
+</instance>
+<instance part="SUPPLY2" gate="G$1" x="7.62" y="38.1" smashed="yes">
+<attribute name="VALUE" x="7.62" y="40.894" size="1.778" layer="96" align="bottom-center"/>
 </instance>
 <instance part="SUPPLY11" gate="G$1" x="127" y="88.9" smashed="yes">
@@
 </instance>
 <instance part="C15" gate="G$1" x="25.4" y="55.88" smashed="yes" rot="R90">
-<attribute name="NAME" x="26.924" y="60.071" size="1.778" layer="95" font="vector" rot="R180"/>
-<attribute name="VALUE" x="23.368" y="58.039" size="1.778" layer="96" font="vector" rot="R180"/>
+<attribute name="NAME" x="30.226" y="58.293" size="1.778" layer="95" font="vector" rot="R180"/>
+<attribute name="VALUE" x="23.368" y="58.293" size="1.778" layer="96" font="vector" rot="R180"/>
 </instance>
 <instance part="C16" gate="G$1" x="25.4" y="50.8" smashed="yes" rot="R90">
@@
 <instance part="D3" gate="G$1" x="25.4" y="132.08" smashed="yes">
 <attribute name="NAME" x="22.86" y="134.112" size="1.778" layer="95" font="vector"/>
-<attribute name="VALUE" x="22.86" y="130.048" size="1.778" layer="96" font="vector" align="top-left"/>
+<attribute name="VALUE" x="10.16" y="130.048" size="1.778" layer="96" font="vector" align="top-left"/>
 </instance>
 <instance part="GND13" gate="1" x="226.06" y="111.76" smashed="yes">
@@
 <instance part="TP6" gate="G$1" x="71.12" y="165.1" smashed="yes">
 <attribute name="NAME" x="70.866" y="166.37" size="1.778" layer="95" font="vector"/>
+</instance>
+<instance part="TP7" gate="G$1" x="152.4" y="134.62" smashed="yes" rot="R90">
+<attribute name="NAME" x="155.194" y="140.97" size="1.778" layer="95" font="vector" rot="R180"/>
+</instance>
+<instance part="TP8" gate="G$1" x="152.4" y="106.68" smashed="yes" rot="R270">
+<attribute name="NAME" x="149.606" y="100.33" size="1.778" layer="95" font="vector"/>
 </instance>
 </instances>
@@
 <segment>
 <pinref part="FB1" gate="G$1" pin="1"/>
-<wire x1="7.62" y1="35.56" x2="7.62" y2="40.64" width="0.1524" layer="91"/>
+<wire x1="7.62" y1="35.56" x2="7.62" y2="38.1" width="0.1524" layer="91"/>
 <pinref part="SUPPLY2" gate="G$1" pin="3.3V"/>
 </segment>
@@
 <pinref part="C2" gate="G$1" pin="2"/>
 <pinref part="GND2" gate="1" pin="GND"/>
-<wire x1="7.62" y1="7.62" x2="7.62" y2="10.16" width="0.1524" layer="91"/>
+<wire x1="7.62" y1="10.16" x2="7.62" y2="12.7" width="0.1524" layer="91"/>
 </segment>
 <segment>
@@
 <segment>
 <pinref part="FB1" gate="G$1" pin="2"/>
-<wire x1="7.62" y1="17.78" x2="7.62" y2="22.86" width="0.1524" layer="91"/>
+<wire x1="7.62" y1="20.32" x2="7.62" y2="22.86" width="0.1524" layer="91"/>
 <pinref part="C2" gate="G$1" pin="1"/>
 <wire x1="7.62" y1="22.86" x2="7.62" y2="25.4" width="0.1524" layer="91"/>
@@
 <segment>
 <pinref part="U4" gate="G$1" pin="SO(D1)"/>
-<wire x1="185.42" y1="68.58" x2="180.34" y2="68.58" width="0.1524" layer="91"/>
-<label x="180.34" y="68.58" size="1.27" layer="95" font="vector" rot="R180" xref="yes"/>
+<wire x1="185.42" y1="68.58" x2="175.26" y2="68.58" width="0.1524" layer="91"/>
+<label x="175.26" y="68.58" size="1.27" layer="95" font="vector" rot="R180" xref="yes"/>
 </segment>
 <segment>
@@
 <segment>
 <pinref part="J3" gate="G$1" pin="2"/>
-<wire x1="147.32" y1="132.08" x2="149.86" y2="132.08" width="0.1524" layer="91"/>
-<label x="149.86" y="132.08" size="1.27" layer="95" font="vector" xref="yes"/>
+<wire x1="147.32" y1="132.08" x2="152.4" y2="132.08" width="0.1524" layer="91"/>
+<label x="154.94" y="132.08" size="1.27" layer="95" font="vector" xref="yes"/>
+<pinref part="TP7" gate="G$1" pin="1"/>
+<wire x1="152.4" y1="132.08" x2="154.94" y2="132.08" width="0.1524" layer="91"/>
+<wire x1="152.4" y1="132.08" x2="152.4" y2="134.62" width="0.1524" layer="91"/>
+<junction x="152.4" y="132.08"/>
 </segment>
 </net>
@@
 <pinref part="J4" gate="G$1" pin="1"/>
 <wire x1="147.32" y1="109.22" x2="152.4" y2="109.22" width="0.1524" layer="91"/>
-<label x="152.4" y="109.22" size="1.27" layer="95" font="vector" xref="yes"/>
-</segment>
-</net>
+<label x="154.94" y="109.22" size="1.27" layer="95" font="vector" xref="yes"/>
+<pinref part="TP8" gate="G$1" pin="1"/>
+<wire x1="152.4" y1="109.22" x2="154.94" y2="109.22" width="0.1524" layer="91"/>
+<wire x1="152.4" y1="106.68" x2="152.4" y2="109.22" width="0.1524" layer="91"/>
+<junction x="152.4" y="109.22"/>
+</segment>
+</net>

Commit message: Adds clarifying text to the 5V and VIN power symbol, changes silk from "VIN" to "3.3V-5V" , and localizes the "OUTPUT" silk better
- Changes DRC to tight with approval of the drill hit errors for better clarification on design choices
Other:
- note added: "3.3-"
- note added: "LEDs"
Changed lines of the file:
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@@
 <wire x1="147.32" y1="35.56" x2="147.32" y2="99.06" width="0.1524" layer="97" style="shortdash"/>
 <wire x1="147.32" y1="99.06" x2="0" y2="99.06" width="0.1524" layer="97" style="shortdash"/>
+<text x="14.224" y="137.414" size="1.778" layer="97">3.3-</text>
+<text x="166.878" y="127.254" size="1.778" layer="97">3.3-</text>
+<text x="78.994" y="142.494" size="1.778" layer="97">LEDs</text>
+<text x="152.654" y="117.094" size="1.778" layer="97">LEDs</text>
 </plain>
 <instances>
